Commit message: Added waist joints to x2 robot training control.

File: resources/robots/x2/urdf/x2_ultra_simple_collision.urdf (robot description, URDF)
Before this commit: robot x2t2.5, 39 links, 38 joints
Joints:
- joint waist_pitch_joint: type fixed -> revolute
- joint waist_roll_joint: type fixed -> revolute
- joint waist_yaw_joint: type fixed -> revolute
