Commit message: Modified x2_fuulbody reward terms to match x2_12dof reward terms.

File: resources/robots/x2/urdf/x2_fullbody.urdf (robot description, URDF)
Before this commit: robot x2t2.5, 39 links, 38 joints
Joints:
- joint left_elbow_joint: origin xyz=0.0140000000488655 0.000199986464082369 -0.0829500000002385 rpy=0 -0.5 0 -> xyz=0.0140000000488655 0.000199986464082369 -0.0829500000002385 rpy=0 0 0
- joint right_elbow_joint: origin xyz=0.0139999999999662 -0.0002000000000143 -0.0829500000000745 rpy=0 -0.5 0 -> xyz=0.0139999999999662 -0.0002000000000143 -0.0829500000000745 rpy=0 0 0
